File: RP2040-PicoProbe.kicad_pcb (KiCad board)
At the start: 4 copper layers, 27.9 x 13.2 mm, 40 parts, among them J1 CONN_UART, J2 CONN_DBG, J5 USB_B_Micro, U1 W25Q128JVS, U2 RP2040, U3 74AUP1T17, U4 W25Q128JVEIQ, U5 MIC5205-3.3YM5, U6 74AUP1T17, Y1 12MHz

Commit message: Moved stuff around
Routing:
- net GND: track 27.5 -> 29.8 mm, vias 39 -> 50
Other:
- outline, holes or cut-outs redrawn
- board text added: "${TITLE}"
Changed lines of the file:
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@@
   (gr_circle (center 139.7 106.934) (end 140.208 106.934)
     (stroke (width 0.15) (type default)) (fill none) (layer "F.SilkS"))
-  (gr_line (start 154.94 94.996) (end 127 94.996)
-    (stroke (width 0.1) (type default)) (layer "Edge.Cuts"))
-  (gr_line (start 154.94 108.204) (end 154.94 94.996)
-    (stroke (width 0.1) (type default)) (layer "Edge.Cuts"))
-  (gr_line (start 127 108.204) (end 154.94 108.204)
-    (stroke (width 0.1) (type default)) (layer "Edge.Cuts"))
-  (gr_line (start 127 94.996) (end 127 108.204)
+  (gr_line (start 153.67 94.996) (end 128.27 94.996)
+    (stroke (width 0.1) (type default)) (layer "Edge.Cuts"))
+  (gr_line (start 153.67 94.996) (end 154.94 96.266)
+    (stroke (width 0.1) (type default)) (layer "Edge.Cuts"))
+  (gr_line (start 128.27 108.204) (end 127 106.934)
+    (stroke (width 0.1) (type default)) (layer "Edge.Cuts"))
+  (gr_line (start 154.94 106.934) (end 154.94 96.266)
+    (stroke (width 0.1) (type default)) (layer "Edge.Cuts"))
+  (gr_line (start 153.67 108.204) (end 154.94 106.934)
+    (stroke (width 0.1) (type default)) (layer "Edge.Cuts"))
+  (gr_line (start 128.27 108.204) (end 153.67 108.204)
+    (stroke (width 0.1) (type default)) (layer "Edge.Cuts"))
+  (gr_line (start 127 96.266) (end 127 106.934)
+    (stroke (width 0.1) (type default)) (layer "Edge.Cuts"))
+  (gr_line (start 128.27 94.996) (end 127 96.266)
     (stroke (width 0.1) (type default)) (layer "Edge.Cuts"))
   (gr_text "5V" (at 152.908 96.52) (layer "B.SilkS")
@@
   )
   (gr_text "GND" (at 152.908 101.6) (layer "B.SilkS")
+    (effects (font (size 1 1) (thickness 0.15)) (justify mirror))
+  )
+  (gr_text "${TITLE}" (at 140.208 101.6) (layer "B.SilkS")
     (effects (font (size 1 1) (thickness 0.15)) (justify mirror))
   )
@@
   )
   (dimension (type aligned) (layer "User.1")
-    (pts (xy 154.94 94.996) (xy 154.94 108.204))
-    (height -12.7)
-    (gr_text "13,2080 mm" (at 166.49 101.6 90) (layer "User.1")
+    (pts (xy 127 94.996) (xy 163.83 94.996))
+    (height -4.826)
+    (gr_text "36,8300 mm" (at 145.415 89.02) (layer "User.1")
+      (effects (font (size 1 1) (thickness 0.15)))
+    )
+    (format (prefix "") (suffix "") (units 3) (units_format 1) (precision 4))
+    (style (thickness 0.15) (arrow_length 1.27) (text_position_mode 0) (extension_height 0.58642) (extension_offset 0.5) keep_text_aligned)
+  )
+  (dimension (type aligned) (layer "User.1")
+    (pts (xy 127 108.204) (xy 127 94.996))
+    (height -6.35)
+    (gr_text "13,2080 mm" (at 119.5 101.6 90) (layer "User.1")
       (effects (font (size 1 1) (thickness 0.15)))
     )
@@
   (segment (start 147.772207 96.880347) (end 147.772207 96.551485) (width 0.2) (layer "B.Cu") (net 1))
   (segment (start 138.424876 106.543124) (end 139.610876 106.543124) (width 0.2) (layer "B.Cu") (net 1))
+  (segment (start 152.816502 100.33) (end 151.892 101.254502) (width 0.2) (layer "F.Cu") (net 2))
   (segment (start 129.911494 102.238805) (end 129.969 102.296311) (width 0.45) (layer "F.Cu") (net 2))
   (segment (start 131.254 102.9) (end 132.558 102.9) (width 0.45) (layer "F.Cu") (net 2))
   (segment (start 143.8995 100.822) (end 144.960314 100.822) (width 0.2) (layer "F.Cu") (net 2))
+  (segment (start 152.885 100.33) (end 152.816502 100.33) (width 0.2) (layer "F.Cu") (net 2))
+  (segment (start 152.885 100.33) (end 152.885 99.428498) (width 0.2) (layer "F.Cu") (net 2))
   (segment (start 145.288 105.156) (end 145.034 104.902) (width 0.2) (layer "F.Cu") (net 2))
   (segment (start 129.911494 102.208412) (end 129.911494 102.238805) (width 0.45) (layer "F.Cu") (net 2))
@@
   (segment (start 145.7705 107.188) (end 145.796 107.188) (width 0.2) (layer "F.Cu") (net 2))
   (segment (start 129.969 102.505) (end 130.364 102.9) (width 0.45) (layer "F.Cu") (net 2))
+  (segment (start 152.885 99.428498) (end 152.908 99.405498) (width 0.2) (layer "F.Cu") (net 2))
   (segment (start 145.7705 97.299682) (end 145.7705 98.044) (width 0.2) (layer "F.Cu") (net 2))
   (segment (start 145.345766 96.874948) (end 145.7705 97.299682) (width 0.2) (layer "F.Cu") (net 2))
@@
   (via (at 142.748 98.0605) (size 0.45) (drill 0.2) (layers "F.Cu" "B.Cu") (net 2))
   (via (at 148.336 99.568) (size 0.45) (drill 0.2) (layers "F.Cu" "B.Cu") (free) (net 2))
+  (via (at 143.256 107.696) (size 0.45) (drill 0.2) (layers "F.Cu" "B.Cu") (free) (net 2))
+  (via (at 140.716 95.504) (size 0.45) (drill 0.2) (layers "F.Cu" "B.Cu") (free) (net 2))
   (via (at 146.304 102.362) (size 0.45) (drill 0.2) (layers "F.Cu" "B.Cu") (free) (net 2))
   (via (at 135.600601 101.017662) (size 0.45) (drill 0.2) (layers "F.Cu" "B.Cu") (free) (net 2))
@@
   (via (at 149.86 99.822) (size 0.45) (drill 0.2) (layers "F.Cu" "B.Cu") (free) (net 2))
   (via (at 145.345766 96.874948) (size 0.45) (drill 0.2) (layers "F.Cu" "B.Cu") (net 2))
+  (via (at 152.908 99.405498) (size 0.45) (drill 0.2) (layers "F.Cu" "B.Cu") (net 2))
   (via (at 146.304 107.696) (size 0.45) (drill 0.2) (layers "F.Cu" "B.Cu") (net 2))
   (via (at 149.086952 107.800653) (size 0.45) (drill 0.2) (layers "F.Cu" "B.Cu") (net 2))
@@
   (via (at 152.908 101.945498) (size 0.45) (drill 0.2) (layers "F.Cu" "B.Cu") (net 2))
   (via (at 150.114 102.87) (size 0.45) (drill 0.2) (layers "F.Cu" "B.Cu") (free) (net 2))
+  (via (at 154.432 101.6) (size 0.45) (drill 0.2) (layers "F.Cu" "B.Cu") (free) (net 2))
   (via (at 141.478 100.838) (size 0.45) (drill 0.2) (layers "F.Cu" "B.Cu") (net 2))
+  (via (at 150.368 95.504) (size 0.45) (drill 0.2) (layers "F.Cu" "B.Cu") (free) (net 2))
   (via (at 134.62 104.843) (size 0.45) (drill 0.2) (layers "F.Cu" "B.Cu") (net 2))
   (via (at 135.636 106.426) (size 0.45) (drill 0.2) (layers "F.Cu" "B.Cu") (net 2))
   (via (at 146.05 99.822) (size 0.45) (drill 0.2) (layers "F.Cu" "B.Cu") (free) (net 2))
   (via (at 137.922 99.822) (size 0.45) (drill 0.2) (layers "F.Cu" "B.Cu") (net 2))
+  (via (at 129.794 107.696) (size 0.45) (drill 0.2) (layers "F.Cu" "B.Cu") (free) (net 2))
   (via (at 141.732 106.68) (size 0.45) (drill 0.2) (layers "F.Cu" "B.Cu") (net 2))
   (via (at 141.732 102.108) (size 0.45) (drill 0.2) (layers "F.Cu" "B.Cu") (net 2))
@@
   (via (at 147.066 99.314) (size 0.45) (drill 0.2) (layers "F.Cu" "B.Cu") (free) (net 2))
   (via (at 141.478 98.806) (size 0.45) (drill 0.2) (layers "F.Cu" "B.Cu") (net 2))
+  (via (at 143.764 103.886) (size 0.45) (drill 0.2) (layers "F.Cu" "B.Cu") (free) (net 2))
+  (via (at 127.508 101.854) (size 0.45) (drill 0.2) (layers "F.Cu" "B.Cu") (free) (net 2))
   (via (at 140.354363 107.737859) (size 0.45) (drill 0.2) (layers "F.Cu" "B.Cu") (net 2))
-  (via (at 130.048 97.282) (size 0.75) (drill 0.45) (layers "F.Cu" "B.Cu") (free) (net 2))
+  (via (at 129.805719 97.279486) (size 0.75) (drill 0.45) (layers "F.Cu" "B.Cu") (free) (net 2))
   (via (at 145.034 104.902) (size 0.45) (drill 0.2) (layers "F.Cu" "B.Cu") (net 2))
+  (via (at 151.384 106.426) (size 0.45) (drill 0.2) (layers "F.Cu" "B.Cu") (free) (net 2))
+  (via (at 130.556 95.504) (size 0.45) (drill 0.2) (layers "F.Cu" "B.Cu") (free) (net 2))
   (via (at 138.43 98.0605) (size 0.45) (drill 0.2) (layers "F.Cu" "B.Cu") (net 2))
+  (via (at 151.892 101.254502) (size 0.45) (drill 0.2) (layers "F.Cu" "B.Cu") (net 2))
   (via (at 149.352 103.886) (size 0.45) (drill 0.2) (layers "F.Cu" "B.Cu") (free) (net 2))
   (via (at 149.760001 97.232276) (size 0.45) (drill 0.2) (layers "F.Cu" "B.Cu") (net 2))
@@
   (segment (start 144.667034 102.756149) (end 144.667034 102.111916) (width 0.2) (layer "B.Cu") (net 36))
   (zone (net 2) (net_name "GND") (layers "F.Cu" "In1.Cu" "B.Cu") (hatch edge 0.5)
-    (connect_pads yes (clearance 0.3))
+    (connect_pads yes (clearance 0.25))
     (min_thickness 0.25) (filled_areas_thickness no)
     (fill yes (thermal_gap 0.5) (thermal_bridge_width 0.5))
@@
   (zone (net 1) (net_name "+3V3") (layer "In2.Cu") (hatch edge 0.5)
     (priority 1)
-    (connect_pads yes (clearance 0.3))
+    (connect_pads yes (clearance 0.25))
     (min_thickness 0.25) (filled_areas_thickness no)
     (fill yes (thermal_gap 0.5) (thermal_bridge_width 0.5))

Commit message: Moved stuff around
Parts:
- moved C17 0.07 mm to (148.1, 104.4)
- moved U3 0.07 mm to (148.1, 106.4)
Routing:
- net +3V3: track 30.8 -> 33.6 mm
Other:
- board text added: "BOOTSEL"
- board text removed: "BOOT"

Commit message: Moved stuff around
Connections:
- U2 pad 2: MCU_TX -> unconnected-(U2-GPIO0-Pad2)
- U2 pad 24: MCU_CLK -> unconnected-(U2-SWCLK-Pad24)
- U2 pad 25: MCU_DIO -> unconnected-(U2-SWD-Pad25)
- U2 pad 3: MCU_RX -> unconnected-(U2-GPIO1-Pad3)
Routing:
- net +3V3: track 33.6 -> 43.8 mm, vias 12 -> 13
- net VUSB: track 29.2 -> 27.9 mm
- net GND: track 29.8 -> 30.0 mm, vias 50 -> 49
