File: RP2040-PicoProbe.kicad_pcb (KiCad board)
At the start: 4 copper layers, 27.9 x 13.2 mm, 40 parts, among them J1 CONN_UART, J2 CONN_DBG, J5 USB_B_Micro, U1 W25Q128JVS, U2 RP2040, U3 74AUP1T17, U4 W25Q128JVEIQ, U5 MIC5205-3.3YM5, U6 74AUP1T17, Y1 12MHz

Commit message: Moved stuff around
Routing:
- net LED_RUN: track 12.9 -> 15.7 mm
- net GND: track 30.0 -> 28.2 mm, vias 49 -> 48
- net LED_RX: track 20.8 -> 21.7 mm
- net +3V3: track 43.8 -> 44.5 mm

Commit message: Moved stuff around
Routing:
- net GND: track 28.2 -> 30.4 mm, vias 48 -> 49
Changed lines of the file:
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@@
   (title_block
     (title "RP2040-PicoProbe-0010")
-    (date "2024-01-14")
+    (date "2024-01-21")
     (rev "1.0")
     (company "(c) 2024 Andriy Golovnya")
@@
     (style (thickness 0.15) (arrow_length 1.27) (text_position_mode 0) (extension_height 0.58642) (extension_offset 0.5) keep_text_aligned)
   )
+  (segment (start 145.815326 98.819) (end 146.210186 98.819) (width 0.2) (layer "F.Cu") (net 1))
   (segment (start 135.89 99.568) (end 135.944 99.622) (width 0.2) (layer "F.Cu") (net 1))
+  (segment (start 146.905814 97.269) (end 147.383554 97.269) (width 0.2) (layer "F.Cu") (net 1))
+  (segment (start 146.558 97.616814) (end 146.905814 97.269) (width 0.2) (layer "F.Cu") (net 1))
   (segment (start 151.335 102.186142) (end 151.335 103.046) (width 0.2) (layer "F.Cu") (net 1))
   (segment (start 147.925186 104.521) (end 147.785186 104.381) (width 0.2) (layer "F.Cu") (net 1))
   (segment (start 137.862 103.2595) (end 137.862 102.72564) (width 0.2) (layer "F.Cu") (net 1))
-  (segment (start 145.136826 99.4975) (end 145.815326 98.819) (width 0.2) (layer "F.Cu") (net 1))
   (segment (start 137.357803 96.3845) (end 137.862 96.3845) (width 0.2) (layer "F.Cu") (net 1))
   (segment (start 142.057815 95.544626) (end 141.768014 95.544626) (width 0.2) (layer "F.Cu") (net 1))
@@
   (segment (start 141.986 104.14) (end 141.80864 104.14) (width 0.2) (layer "F.Cu") (net 1))
   (segment (start 153.309803 104.975197) (end 152.885 105.4) (width 0.2) (layer "F.Cu") (net 1))
-  (segment (start 146.210186 98.819) (end 146.558 98.471186) (width 0.2) (layer "F.Cu") (net 1))
   (segment (start 138.06564 102.522) (end 141.25836 102.522) (width 0.2) (layer "F.Cu") (net 1))
   (segment (start 151.672002 101.84914) (end 151.335 102.186142) (width 0.2) (layer "F.Cu") (net 1))
@@
   (segment (start 145.012326 99.622) (end 143.8995 99.622) (width 0.2) (layer "F.Cu") (net 1))
   (segment (start 146.558 98.471186) (end 146.558 97.616814) (width 0.2) (layer "F.Cu") (net 1))
+  (segment (start 147.383554 97.269) (end 147.772207 96.880347) (width 0.2) (layer "F.Cu") (net 1))
   (segment (start 137.0245 97.622) (end 137.0245 97.222) (width 0.2) (layer "F.Cu") (net 1))
   (segment (start 137.022696 96.049393) (end 137.0245 96.051197) (width 0.2) (layer "F.Cu") (net 1))
@@
   (segment (start 153.309803 104.485498) (end 153.309803 104.975197) (width 0.2) (layer "F.Cu") (net 1))
   (segment (start 137.0245 96.051197) (end 137.0245 97.222) (width 0.2) (layer "F.Cu") (net 1))
+  (segment (start 146.210186 98.819) (end 146.558 98.471186) (width 0.2) (layer "F.Cu") (net 1))
   (segment (start 152.885 106.311502) (end 152.885 105.4) (width 0.2) (layer "F.Cu") (net 1))
   (segment (start 151.335 103.046) (end 149.86 104.521) (width 0.2) (layer "F.Cu") (net 1))
-  (segment (start 147.294467 96.880347) (end 147.772207 96.880347) (width 0.2) (layer "F.Cu") (net 1))
-  (segment (start 146.558 97.616814) (end 147.294467 96.880347) (width 0.2) (layer "F.Cu") (net 1))
+  (segment (start 145.136826 99.4975) (end 145.815326 98.819) (width 0.2) (layer "F.Cu") (net 1))
   (segment (start 141.80864 104.14) (end 141.462 103.79336) (width 0.2) (layer "F.Cu") (net 1))
   (segment (start 149.86 104.521) (end 147.925186 104.521) (width 0.2) (layer "F.Cu") (net 1))
   (segment (start 135.944 99.622) (end 137.0245 99.622) (width 0.2) (layer "F.Cu") (net 1))
   (segment (start 137.022696 96.049393) (end 137.357803 96.3845) (width 0.2) (layer "F.Cu") (net 1))
-  (segment (start 145.815326 98.819) (end 146.210186 98.819) (width 0.2) (layer "F.Cu") (net 1))
   (via (at 140.462 105.664) (size 0.45) (drill 0.2) (layers "F.Cu" "B.Cu") (net 1))
   (via (at 151.672002 101.84914) (size 0.45) (drill 0.2) (layers "F.Cu" "B.Cu") (net 1))
@@
   (segment (start 131.254 102.9) (end 132.558 102.9) (width 0.45) (layer "F.Cu") (net 2))
   (segment (start 130.048402 102.584402) (end 130.364 102.9) (width 0.45) (layer "F.Cu") (net 2))
+  (segment (start 129.969 103.174) (end 129.969 104.681619) (width 0.45) (layer "F.Cu") (net 2))
   (segment (start 143.8995 100.822) (end 144.960314 100.822) (width 0.2) (layer "F.Cu") (net 2))
   (segment (start 130.048402 102.044146) (end 130.048402 102.584402) (width 0.45) (layer "F.Cu") (net 2))
@@
   (segment (start 129.943158 101.938902) (end 130.048402 102.044146) (width 0.45) (layer "F.Cu") (net 2))
   (segment (start 146.304 107.696) (end 145.796 107.188) (width 0.2) (layer "F.Cu") (net 2))
+  (segment (start 130.243 102.9) (end 129.969 103.174) (width 0.45) (layer "F.Cu") (net 2))
   (segment (start 145.288 105.156) (end 145.034 104.902) (width 0.2) (layer "F.Cu") (net 2))
   (segment (start 145.7705 96.810612) (end 145.7705 98.044) (width 0.2) (layer "F.Cu") (net 2))
@@
   (segment (start 141.494 100.822) (end 141.478 100.838) (width 0.2) (layer "F.Cu") (net 2))
   (segment (start 144.960314 100.822) (end 146.304 102.165686) (width 0.2) (layer "F.Cu") (net 2))
+  (segment (start 130.364 102.9) (end 130.243 102.9) (width 0.45) (layer "F.Cu") (net 2))
   (segment (start 135.1535 106.9085) (end 135.636 106.426) (width 0.2) (layer "F.Cu") (net 2))
+  (segment (start 129.969 104.681619) (end 129.819002 104.831617) (width 0.45) (layer "F.Cu") (net 2))
   (segment (start 135.128 96.012) (end 134.62 95.504) (width 0.2) (layer "F.Cu") (net 2))
   (segment (start 146.304 102.165686) (end 146.304 102.362) (width 0.2) (layer "F.Cu") (net 2))
@@
   (via (at 140.462 99.822) (size 0.45) (drill 0.2) (layers "F.Cu" "B.Cu") (net 2))
   (via (at 139.446 100.838) (size 0.45) (drill 0.2) (layers "F.Cu" "B.Cu") (net 2))
+  (via (at 129.819002 104.831617) (size 0.75) (drill 0.45) (layers "F.Cu" "B.Cu") (net 2))
   (via (at 136.398 103.632) (size 0.45) (drill 0.2) (layers "F.Cu" "B.Cu") (free) (net 2))
   (via (at 142.748 98.0605) (size 0.45) (drill 0.2) (layers "F.Cu" "B.Cu") (net 2))
@@
   (segment (start 150.331463 106.951) (end 149.363988 106.951) (width 0.2) (layer "In2.Cu") (net 18))
   (segment (start 142.06564 102.522) (end 141.862 102.72564) (width 0.2) (layer "F.Cu") (net 19))
-  (segment (start 149.608 95.875177) (end 149.232321 95.499498) (width 0.2) (layer "F.Cu") (net 19))
   (segment (start 141.862 102.72564) (end 141.862 103.2595) (width 0.2) (layer "F.Cu") (net 19))
+  (segment (start 149.608 95.875177) (end 149.232321 95.499498) (width 0.2) (layer "F.Cu") (net 19))
+  (segment (start 143.039595 101.719057) (end 143.039595 102.070405) (width 0.2) (layer "F.Cu") (net 19))
+  (segment (start 143.039595 102.070405) (end 142.588 102.522) (width 0.2) (layer "F.Cu") (net 19))
+  (segment (start 142.588 102.522) (end 142.06564 102.522) (width 0.2) (layer "F.Cu") (net 19))
   (segment (start 149.608 96.012) (end 149.608 95.875177) (width 0.2) (layer "F.Cu") (net 19))
-  (segment (start 142.236652 102.522) (end 142.06564 102.522) (width 0.2) (layer "F.Cu") (net 19))
-  (segment (start 143.039595 101.719057) (end 142.236652 102.522) (width 0.2) (layer "F.Cu") (net 19))
   (via (at 149.232321 95.499498) (size 0.45) (drill 0.2) (layers "F.Cu" "B.Cu") (net 19))
   (via (at 143.039595 101.719057) (size 0.45) (drill 0.2) (layers "F.Cu" "B.Cu") (net 19))
